Commit message: update yr_lle_sim: update xacro to add hip_abd joint/link to rviz model, add STL meshes

File: src/yr_lle_sim/urdf/exo.xacro (robot description, xacro)
@@ -6,23 +6,40 @@
     <!-- LINKS                                                   -->
     <!-- ======================================================= -->
-    <xacro:create_link name="waist_link" m="${waist_m}" l="${waist_l}"
-        w="${waist_w}" h="${waist_h}" mat="${waist_mat}" />
+    <!-- <xacro:create_link name="waist_link" m="${waist_m}" l="${waist_l}"
+        w="${waist_w}" h="${waist_h}" mat="${waist_mat}" /> -->
+    <xacro:create_link2 name="waist_link" m="${waist_m}" l="${waist_l}" w="${waist_w}"
+        h="${waist_h}" o_x="0" o_y="${waist_mesh_w/2}" o_z="${-waist_h_offset}" o_r="0" o_p="${-PI}"
+        o_yaw="${-PI}"
+        mat="${waist_mat}"
+        mesh_filename="${waist_mesh}" mirror="1" />
+    <!-- <xacro:create_link2 name="l_pel_link" m="${pel_m}" l="${pel_l}"
+    w="${pel_w}"
+        h="${pel_h}" o_x="0" o_y="${waist_w/2}" o_z="0" o_r="0" o_p="0"
+        o_yaw="${PI/2}" mat="${pel_mat}" mesh_filename="${pel_mesh}" mirror="1" /> -->
+    <xacro:create_link2 name="l_pel_link" m="${pel_m}" l="${pel_l}" w="${pel_w}"
+        h="${pel_h}" o_x="${pel_x_offset}" o_y="${pel_y_offset}"
+        o_z="${-pel_h_offset}" o_r="0.0" o_p="0"
+        o_yaw="0" mat="${pel_mat}" mesh_filename="${pel_mesh}" mirror="1" />
     <xacro:create_link2 name="l_thigh_link" m="${thigh_m}" l="${thigh_l}" w="${thigh_w}"
         h="${thigh_h}" o_x="${thigh_w}" o_y="${thigh_w/2}" o_z="${-thigh_l}" o_r="0" o_p="0"
         o_yaw="${PI}" mat="${thigh_mat}" mesh_filename="${thigh_mesh}" mirror="1" />
-    <xacro:create_link2 name="l_calf_link" m="${calf_m}" l="${calf_l}" w="${calf_w}"
-        h="${calf_h}" o_x="${calf_w}" o_y="${calf_w/2}" o_z="${-calf_l}" o_r="0" o_p="0"
+    <xacro:create_link2 name="l_shank_link" m="${shank_m}" l="${shank_l}" w="${shank_w}"
+        h="${shank_h}" o_x="${shank_w}" o_y="${shank_w/2}" o_z="${-shank_l}" o_r="0" o_p="0"
         o_yaw="${PI}"
-        mat="${calf_mat}" mesh_filename="${shank_mesh}" mirror="1" />
+        mat="${shank_mat}" mesh_filename="${shank_mesh}" mirror="1" />
     <xacro:create_link2 name="l_foot_link" m="${foot_m}" l="${foot_l}" w="${foot_w}"
         h="${foot_h}" o_x="${-foot_h}" o_y="${foot_w}" o_z="${-foot_l}" o_r="0" o_p="0" o_yaw="0"
         mat="${foot_mat}"
         mesh_filename="${foot_mesh}" mirror="-1" />
+    <xacro:create_link2 name="r_pel_link" m="${pel_m}" l="${pel_l}" w="${pel_w}"
+        h="${pel_h}" o_x="${pel_x_offset}" o_y="${pel_y_offset}"
+        o_z="${-pel_h_offset}" o_r="0" o_p="0"
+        o_yaw="0" mat="${pel_mat}" mesh_filename="${pel_mesh}" mirror="1" />
     <xacro:create_link2 name="r_thigh_link" m="${thigh_m}" l="${thigh_l}" w="${thigh_w}"
         h="${thigh_h}" o_x="${-thigh_w}" o_y="${-thigh_w/2}" o_z="${-thigh_l}" o_r="0" o_p="0"
         o_yaw="0" mat="${thigh_mat}" mesh_filename="${thigh_mesh}" mirror="1" />
-    <xacro:create_link2 name="r_calf_link" m="${calf_m}" l="${calf_l}" w="${calf_w}"
-        h="${calf_h}" o_x="${-calf_w}" o_y="${-calf_w/2}" o_z="${-calf_l}" o_r="0" o_p="0" o_yaw="0"
-        mat="${calf_mat}" mesh_filename="${shank_mesh}" mirror="1" />
+    <xacro:create_link2 name="r_shank_link" m="${shank_m}" l="${shank_l}" w="${shank_w}"
+        h="${shank_h}" o_x="${-shank_w}" o_y="${-shank_w/2}" o_z="${-shank_l}" o_r="0" o_p="0" o_yaw="0"
+        mat="${shank_mat}" mesh_filename="${shank_mesh}" mirror="1" />
     <xacro:create_link2 name="r_foot_link" m="${foot_m}" l="${foot_l}" w="${foot_w}"
         h="${foot_h}" o_x="${-foot_h}" o_y="${-foot_w}" o_z="${-foot_l}" o_r="0" o_p="0" o_yaw="0"
@@ -33,21 +50,35 @@
     <!-- ======================================================= -->
     <xacro:macro name="create_leg" params="side origin_y">
-        <xacro:create_joint name="${side}_hip_joint" parent="waist_link" child="${side}_thigh_link"
+        <!-- origin_y="${origin_y}" -->
+        <xacro:create_joint name="${side}_pel_joint" parent="waist_link"
+            child="${side}_pel_link" origin_x="0" origin_y="${origin_y}"
+            origin_z="0" o_roll="0"
+            o_pitch="0" o_yaw="0"
+            axis_x="1" axis_y="0" axis_z="0"
+            lower_limit="-1.5" upper_limit="1.5" effort="1000" velocity="10.0" />
+        <xacro:create_joint name="${side}_hip_joint" parent="${side}_pel_link"
+            child="${side}_thigh_link"
+            origin_x="0" origin_y="0" origin_z="${-pel_l}" o_roll="0" o_pitch="0" o_yaw="0"
+            axis_x="0" axis_y="1" axis_z="0"
+            lower_limit="-${PI}" upper_limit="${PI}" effort="100000" velocity="100.0" />
+        <!-- <xacro:create_joint name="${side}_hip_joint" parent="waist_link"
+        child="${side}_thigh_link"
             origin_x="0" origin_y="${origin_y}" origin_z="0" o_roll="0" o_pitch="0" o_yaw="0"
             axis_x="0" axis_y="1" axis_z="0"
-            lower_limit="-${PI}" upper_limit="${PI}" effort="100000" velocity="100.0" />
-        <xacro:create_joint name="${side}_knee_joint" parent="${side}_thigh_link"
-            child="${side}_calf_link"
+            lower_limit="-${PI}" upper_limit="${PI}" effort="100000" velocity="100.0" /> -->
+        <xacro:create_joint name="${side}_kne_joint" parent="${side}_thigh_link"
+            child="${side}_shank_link"
             origin_x="0" origin_y="0" origin_z="${-thigh_l}" o_roll="0" o_pitch="0" o_yaw="0"
             axis_x="0" axis_y="1" axis_z="0"
             lower_limit="-${PI}" upper_limit="${PI}" effort="100000" velocity="100.0" />
-        <xacro:create_joint name="${side}_ankle_joint" parent="${side}_calf_link"
+        <xacro:create_joint name="${side}_ank_joint" parent="${side}_shank_link"
             child="${side}_foot_link"
-            origin_x="0" origin_y="0" origin_z="${-calf_l}" o_roll="0" o_pitch="${-PI/2}" o_yaw="0"
+            origin_x="0" origin_y="0" origin_z="${-shank_l}" o_roll="0" o_pitch="${-PI/2}" o_yaw="0"
             axis_x="0" axis_y="1" axis_z="0"
             lower_limit="-1.75" upper_limit="1.75" effort="1000" velocity="10.0" />
     </xacro:macro>
-    <xacro:create_leg side="l" origin_y="${waist_w / 2}" />
-    <xacro:create_leg side="r" origin_y="${-waist_w / 2}" />
+    <xacro:property name="waist_w_offset" value="${waist_w * 0.42}" />
+    <xacro:create_leg side="l" origin_y="${waist_w_offset}" />
+    <xacro:create_leg side="r" origin_y="${-waist_w_offset}" />
     <!-- ======================================================= -->
     <!-- GAZEBO                                                  -->
@@ -68,5 +99,5 @@
             <stateInterface>effort</stateInterface>
         </joint>
-        <joint name="l_knee_joint">
+        <joint name="l_kne_joint">
             <commandInterface>effort</commandInterface>
             <stateInterface>position</stateInterface>
@@ -78,11 +109,11 @@
         <material>Gazebo/Blue</material>
     </gazebo>
-    <gazebo reference="l_calf_link">
+    <gazebo reference="l_shank_link">
         <material>Gazebo/Green</material>
     </gazebo>
     <xacro:macro name="create_leg_transmissions" params="side">
         <xacro:create_transmission joint_name="${side}_hip_joint" />
-        <xacro:create_transmission joint_name="${side}_knee_joint" />
-        <!-- <xacro:create_transmission joint_name="${side}_ankle_joint" /> -->
+        <xacro:create_transmission joint_name="${side}_kne_joint" />
+        <!-- <xacro:create_transmission joint_name="${side}_ank_joint" /> -->
     </xacro:macro>
     <!-- <xacro:create_leg_transmissions side="l" />

File: src/yr_lle_sim/urdf/model_gazebo.xacro (robot description, xacro)
@@ -25,8 +25,8 @@
         h="${thigh_h}" o_x="${thigh_w}" o_y="${thigh_w/2}" o_z="${-thigh_l}" o_r="0" o_p="0"
         o_yaw="${PI}" mat="${thigh_mat}" mesh_filename="${thigh_mesh}" mirror="1" />
-    <xacro:create_link2 name="l_calf_link" m="${calf_m}" l="${calf_l}" w="${calf_w}"
-        h="${calf_h}" o_x="${calf_w}" o_y="${calf_w/2}" o_z="${-calf_l}" o_r="0" o_p="0"
+    <xacro:create_link2 name="l_shank_link" m="${shank_m}" l="${shank_l}" w="${shank_w}"
+        h="${shank_h}" o_x="${shank_w}" o_y="${shank_w/2}" o_z="${-shank_l}" o_r="0" o_p="0"
         o_yaw="${PI}"
-        mat="${calf_mat}" mesh_filename="${shank_mesh}" mirror="1" />
+        mat="${shank_mat}" mesh_filename="${shank_mesh}" mirror="1" />
     <xacro:create_link2 name="l_foot_link" m="${foot_m}" l="${foot_l}" w="${foot_w}"
         h="${foot_h}" o_x="${-foot_h}" o_y="${foot_w}" o_z="${-foot_l}" o_r="0" o_p="0" o_yaw="0"
@@ -36,7 +36,7 @@
         h="${thigh_h}" o_x="${-thigh_w}" o_y="${-thigh_w/2}" o_z="${-thigh_l}" o_r="0" o_p="0"
         o_yaw="0" mat="${thigh_mat}" mesh_filename="${thigh_mesh}" mirror="1" />
-    <xacro:create_link2 name="r_calf_link" m="${calf_m}" l="${calf_l}" w="${calf_w}"
-        h="${calf_h}" o_x="${-calf_w}" o_y="${-calf_w/2}" o_z="${-calf_l}" o_r="0" o_p="0" o_yaw="0"
-        mat="${calf_mat}" mesh_filename="${shank_mesh}" mirror="1" />
+    <xacro:create_link2 name="r_shank_link" m="${shank_m}" l="${shank_l}" w="${shank_w}"
+        h="${shank_h}" o_x="${-shank_w}" o_y="${-shank_w/2}" o_z="${-shank_l}" o_r="0" o_p="0" o_yaw="0"
+        mat="${shank_mat}" mesh_filename="${shank_mesh}" mirror="1" />
     <xacro:create_link2 name="r_foot_link" m="${foot_m}" l="${foot_l}" w="${foot_w}"
         h="${foot_h}" o_x="${-foot_h}" o_y="${-foot_w}" o_z="${-foot_l}" o_r="0" o_p="0" o_yaw="0"
@@ -51,12 +51,12 @@
             axis_x="0" axis_y="1" axis_z="0"
             lower_limit="-${PI}" upper_limit="${PI}" effort="100000" velocity="100.0" />
-        <xacro:create_joint name="${side}_knee_joint" parent="${side}_thigh_link"
-            child="${side}_calf_link"
+        <xacro:create_joint name="${side}_kne_joint" parent="${side}_thigh_link"
+            child="${side}_shank_link"
             origin_x="0" origin_y="0" origin_z="${-thigh_l}" o_roll="0" o_pitch="0" o_yaw="0"
             axis_x="0" axis_y="1" axis_z="0"
             lower_limit="-${PI}" upper_limit="${PI}" effort="100000" velocity="100.0" />
-        <xacro:create_joint name="${side}_ankle_joint" parent="${side}_calf_link"
+        <xacro:create_joint name="${side}_ank_joint" parent="${side}_shank_link"
             child="${side}_foot_link"
-            origin_x="0" origin_y="0" origin_z="${-calf_l}" o_roll="0" o_pitch="${-PI/2}" o_yaw="0"
+            origin_x="0" origin_y="0" origin_z="${-shank_l}" o_roll="0" o_pitch="${-PI/2}" o_yaw="0"
             axis_x="0" axis_y="1" axis_z="0"
             lower_limit="-1.75" upper_limit="1.75" effort="1000" velocity="10.0" />
@@ -82,5 +82,5 @@
             <stateInterface>effort</stateInterface>
         </joint>
-        <joint name="l_knee_joint">
+        <joint name="l_kne_joint">
             <commandInterface>effort</commandInterface>
             <stateInterface>position</stateInterface>
@@ -91,6 +91,6 @@
     <xacro:define_gazebo_material link_name="l_thigh_link" r="0.7" g="0.7" b="0.7" a="1" />
     <xacro:define_gazebo_material link_name="r_thigh_link" r="0.7" g="0.7" b="0.7" a="1" />
-    <xacro:define_gazebo_material link_name="l_calf_link" r="0.8" g="0.8" b="0.8" a="1" />
-    <xacro:define_gazebo_material link_name="r_calf_link" r="0.8" g="0.8" b="0.8" a="1" />
+    <xacro:define_gazebo_material link_name="l_shank_link" r="0.8" g="0.8" b="0.8" a="1" />
+    <xacro:define_gazebo_material link_name="r_shank_link" r="0.8" g="0.8" b="0.8" a="1" />
     <xacro:define_gazebo_material link_name="l_foot_link" r="0.7" g="0.7" b="0.7" a="1" />
     <xacro:define_gazebo_material link_name="r_foot_link" r="0.7" g="0.7" b="0.7" a="1" />
@@ -100,6 +100,6 @@
     <xacro:macro name="create_leg_transmissions" params="side">
         <xacro:create_transmission joint_name="${side}_hip_joint" />
-        <xacro:create_transmission joint_name="${side}_knee_joint" />
-        <!-- <xacro:create_transmission joint_name="${side}_ankle_joint" /> -->
+        <xacro:create_transmission joint_name="${side}_kne_joint" />
+        <!-- <xacro:create_transmission joint_name="${side}_ank_joint" /> -->
     </xacro:macro>
     <!-- <xacro:create_leg_transmissions side="l" />
@@ -156,6 +156,6 @@
     <xacro:add_imu_sensor link_name="l_thigh_link" />
     <xacro:add_imu_sensor link_name="r_thigh_link" />
-    <xacro:add_imu_sensor link_name="l_calf_link" />
-    <xacro:add_imu_sensor link_name="r_calf_link" />
+    <xacro:add_imu_sensor link_name="l_shank_link" />
+    <xacro:add_imu_sensor link_name="r_shank_link" />
     <xacro:add_imu_sensor link_name="l_foot_link" />
     <xacro:add_imu_sensor link_name="r_foot_link" />

File: src/yr_lle_sim/urdf/properties.xacro (robot description, xacro)
@@ -2,5 +2,5 @@
 <robot name="lower_limb_exoskeleton" xmlns:xacro="http://www.ros.org/wiki/xacro">
     <xacro:property name="PI" value="3.1415926535897931" />
-    <xacro:property name="alpha" value="0.8" />
+    <xacro:property name="alpha" value="1.0" />
     <material name="silver">
         <color rgba="0.8 0.8 0.8 ${alpha}" />
@@ -12,20 +12,34 @@
         <color rgba="0.8 0.8 1 ${alpha}" />
     </material>
-    <xacro:property name="waist_m" value="1" />
+    <xacro:property name="waist_m" value="2.0" />
     <xacro:property name="waist_l" value="0.05" />
-    <xacro:property name="waist_w" value="0.35" />
     <xacro:property name="waist_h" value="0.05" />
     <xacro:property name="waist_mat" value="silver" />
-    <xacro:property name="thigh_m" value="1" />
+    <xacro:property name="waist_mesh_w" value="0.42" />
+    <xacro:property name="waist_w" value="${waist_mesh_w}" />
+    <xacro:property name="waist_h_offset" value="0.062" />
+    <xacro:property name="waist_mesh"
+        value="file://$(find yr_lle_sim)/urdf/meshes_yr/waist_center.STL" />
+    <xacro:property name="pel_m" value="1.0" />
+    <xacro:property name="pel_l" value="0.0" />
+    <xacro:property name="pel_w" value="0.0" />
+    <xacro:property name="pel_h" value="0.0" />
+    <xacro:property name="pel_mat" value="silver" />
+    <xacro:property name="pel_x_offset" value="-0.09" />
+    <xacro:property name="pel_y_offset" value="-0.028" />
+    <xacro:property name="pel_h_offset" value="0.088" />
+    <xacro:property name="pel_mesh"
+        value="file://$(find yr_lle_sim)/urdf/meshes_yr/orig.waist_corner_bracket.STL" />
+    <xacro:property name="thigh_m" value="1.5" />
     <xacro:property name="thigh_l" value="0.468" />
     <xacro:property name="thigh_w" value="0.1" />
     <xacro:property name="thigh_h" value="0.1" />
     <xacro:property name="thigh_mat" value="blue" />
-    <xacro:property name="calf_m" value="1" />
-    <xacro:property name="calf_l" value="0.468" />
-    <xacro:property name="calf_w" value="0.1" />
-    <xacro:property name="calf_h" value="0.1" />
-    <xacro:property name="calf_mat" value="green" />
-    <xacro:property name="foot_m" value="1" />
+    <xacro:property name="shank_m" value="1.5" />
+    <xacro:property name="shank_l" value="0.468" />
+    <xacro:property name="shank_w" value="0.1" />
+    <xacro:property name="shank_h" value="0.1" />
+    <xacro:property name="shank_mat" value="green" />
+    <xacro:property name="foot_m" value="1.0" />
     <xacro:property name="foot_l" value="0.15" />
     <xacro:property name="foot_w" value="0.08" />
