Commit message: update README.md, add gazebo launch/xacro files

File: src/yr_lle_sim/urdf/macros.xacro (robot description, xacro)
@@ -114,8 +114,50 @@
         </transmission>
     </xacro:macro>
-    <!-- <commandInterface name="position"> -->
-    <!-- <commandInterface name="effort">
-                <param name="min">-2000</param>
-                <param name="max">2000</param>
-            </commandInterface> -->
+    <xacro:macro name="set_gazebo_material" params="link_name material">
+        <gazebo reference="${link_name}">
+            <material>${material}</material>
+        </gazebo>
+    </xacro:macro>
+    <xacro:macro name="define_gazebo_material" params="link_name r g b a">
+        <gazebo reference="${link_name}">
+            <material>Gazebo/White</material>
+            <visual>
+                <material>
+                    <ambient>${r} ${g} ${b} ${a}</ambient>
+                    <diffuse>${r} ${g} ${b} ${a}</diffuse>
+                    <specular>0.1 0.1 0.1 1</specular>
+                    <emissive>0 0 0 0</emissive>
+                </material>
+            </visual>
+        </gazebo>
+    </xacro:macro>
+    <xacro:macro name="add_imu_sensor" params="link_name">
+        <gazebo reference="${link_name}">
+            <sensor type="imu" name="${link_name}_imu_sensor">
+                <always_on>true</always_on>
+                <update_rate>50</update_rate>
+                <imu>
+                    <angular_velocity>
+                        <x>0.0</x>
+                        <y>0.0</y>
+                        <z>0.0</z>
+                    </angular_velocity>
+                    <linear_acceleration>
+                        <x>0.0</x>
+                        <y>0.0</y>
+                        <z>0.0</z>
+                    </linear_acceleration>
+                </imu>
+                <plugin name="gazebo_ros_imu_controller" filename="libgazebo_ros_imu_sensor.so">
+                    <ros>
+                        <!-- Output topic name -->
+                        <namespace>${link_name}</namespace>
+                        <argument>imu/data:=imu</argument>
+                    </ros>
+                    <!-- Frame ID for the IMU data -->
+                    <frameName>${link_name}</frameName>
+                </plugin>
+            </sensor>
+        </gazebo>
+    </xacro:macro>
 </robot>

File: src/yr_lle_sim/urdf/properties.xacro (robot description, xacro)
@@ -21,6 +21,4 @@
     <xacro:property name="thigh_w" value="0.1" />
     <xacro:property name="thigh_h" value="0.1" />
-    <!-- <xacro:property name="thigh_w" value="0.0657" />
-    <xacro:property name="thigh_h" value="0.0819" /> -->
     <xacro:property name="thigh_mat" value="blue" />
     <xacro:property name="calf_m" value="1" />
@@ -30,14 +28,15 @@
     <xacro:property name="calf_mat" value="green" />
     <xacro:property name="foot_m" value="1" />
-    <xacro:property name="foot_l" value="0.15" /> <!-- distance down from shank link -->
-    <xacro:property name="foot_w" value="0.08" /> <!-- same direction as waist expand -->
-    <xacro:property name="foot_h" value="0.10" /> <!-- back/forward -->
+    <xacro:property name="foot_l" value="0.15" />
+    <xacro:property name="foot_w" value="0.08" />
+    <xacro:property name="foot_h" value="0.10" />
     <xacro:property name="foot_mat" value="silver" />
-    <xacro:property name="thigh_mesh" value="package://yr_lle_sim/urdf/meshes_yr/exo_thigh.STL" />
-    <xacro:property name="shank_mesh" value="package://yr_lle_sim/urdf/meshes_yr/exo_shank.STL" />
-    <xacro:property name="foot_mesh" value="package://yr_lle_sim/urdf/meshes_yr/exo_foot.STL" />
-    <!-- <xacro:property name="thigh_mesh"
-    value="package://yr_lle_sim/urdf/meshes/front_left_upper_leg.dae" />
-    <xacro:property name="thigh_mesh"
-    value="package://yr_lle_sim/urdf/meshes/front_right_lower_leg.dae" /> -->
+    <xacro:property name="stand_base_width" value="0.5" />
+    <xacro:property name="stand_base_depth" value="0.5" />
+    <xacro:property name="stand_base_height" value="0.05" />
+    <xacro:property name="pole_height" value="1.2" />
+    <xacro:property name="pole_radius" value="0.02" />
+    <xacro:property name="thigh_mesh" value="file://$(find yr_lle_sim)/urdf/meshes_yr/exo_thigh.STL" />
+    <xacro:property name="shank_mesh" value="file://$(find yr_lle_sim)/urdf/meshes_yr/exo_shank.STL" />
+    <xacro:property name="foot_mesh" value="file://$(find yr_lle_sim)/urdf/meshes_yr/exo_foot.STL" />
 </robot>

Commit message: first commit

File: src/yr_lle_sim/urdf/macros.xacro (robot description, xacro)
@@ -42,8 +42,27 @@
         <link name="${name}">
             <collision>
+                <!-- <origin xyz="0 0 ${-l/2}" rpy="0 0 0" />
+                <geometry>
+                    <box size="${h} ${w} ${l}" />
+                </geometry> -->
+                <xacro:if value="${mesh_filename != ''}">
+                    <!-- <origin xyz="0 0 0" rpy="0 0 ${-PI}" /> -->
+                    <!-- <origin xyz="${-h} ${-w/2} ${-l}" rpy="${PI/2} 0 ${PI/2 + float(o_yaw)}" /> -->
+                    <origin xyz="${o_x} ${o_y} ${o_z}" rpy="${PI/2} 0 ${PI/2 + o_yaw}" />
+                </xacro:if>
+                <xacro:unless value="${mesh_filename != ''}">
+                    <origin xyz="0 0 ${-l/2}" rpy="0 0 ${-PI}" />
+                </xacro:unless>
+                <geometry>
+                    <xacro:if value="${mesh_filename != ''}">
+                        <mesh filename="${mesh_filename}"
+                            scale="${mirror*mesh_scale} ${mesh_scale} ${mesh_scale}" />
+                    </xacro:if>
+                    <xacro:unless value="${mesh_filename != ''}">
+                        <box size="${h} ${w} ${l}" />
+                    </xacro:unless>
+                </geometry>
                 <origin xyz="0 0 ${-l/2}" rpy="0 0 0" />
-                <geometry>
-                    <box size="${l} ${w} ${h}" />
-                </geometry>
+                <material name="${mat}" />
             </collision>
             <visual>
@@ -99,4 +118,13 @@
         </joint>
     </xacro:macro>
+    <xacro:macro name="create_joint2"
+        params="name parent child origin_x origin_y origin_z o_roll o_pitch o_yaw axis_x axis_y axis_z lower_limit upper_limit effort velocity">
+        <joint name="${name}" type="continuous">
+            <parent link="${parent}" />
+            <child link="${child}" />
+            <origin xyz="${origin_x} ${origin_y} ${origin_z}" rpy="${o_roll} ${o_pitch} ${o_yaw}" />
+            <axis xyz="${axis_x} ${axis_y} ${axis_z}" />
+        </joint>
+    </xacro:macro>
     <!-- ======================================================= -->
     <!-- TRANSMISSION                                            -->
@@ -132,7 +160,8 @@
         </gazebo>
     </xacro:macro>
-    <xacro:macro name="add_imu_sensor" params="link_name">
+    <xacro:macro name="add_imu_sensor" params="link_name joint_name">
         <gazebo reference="${link_name}">
             <sensor type="imu" name="${link_name}_imu_sensor">
+                <pose>0 0 0 0 0 0</pose>
                 <always_on>true</always_on>
                 <update_rate>50</update_rate>
@@ -149,9 +178,9 @@
                     </linear_acceleration>
                 </imu>
-                <plugin name="gazebo_ros_imu_controller" filename="libgazebo_ros_imu_sensor.so">
+                <plugin name="imu" filename="libgazebo_ros_imu_sensor.so">
                     <ros>
                         <!-- Output topic name -->
-                        <namespace>${link_name}</namespace>
-                        <argument>imu/data:=imu</argument>
+                        <namespace>${joint_name}</namespace>
+                        <argument>imu/out:=imu</argument>
                     </ros>
                     <!-- Frame ID for the IMU data -->
