Commit message: first commit

File: src/yr_lle_sim/urdf/model_gazebo.xacro (robot description, xacro)
@@ -1,162 +1,314 @@
 <?xml version="1.0"?>
 <robot name="lower_limb_exoskeleton" xmlns:xacro="http://www.ros.org/wiki/xacro">
-    <xacro:include filename="properties.xacro" />
-    <xacro:include filename="macros.xacro" />
-    <!-- <xacro:property name="thigh_mesh" value="" />
-    <xacro:property name="shank_mesh" value="" />
-    <xacro:property name="foot_mesh" value="" /> -->
-    <!-- <xacro:property name="thigh_mesh" value="package://yr_lle_sim/urdf/meshes_yr/exo_thigh.dae"
-    /> -->
-    <!-- <xacro:property name="thigh_mesh"
-    value="/home/user/gitlab/yr-soc-ws/ros-ws/src/yr_lle_sim/urdf/meshes_yr/exo_thigh.dae" /> -->
-    <!-- <xacro:property name="thigh_mesh"
-    value="/home/user/gitlab/yr-soc-ws/ros-ws/src/yr_lle_sim/urdf/meshes_yr/exo_thigh.STL" /> -->
-    <!-- <xacro:property name="thigh_mesh" value="file://$(find
-    yr_lle_sim)/urdf/meshes_yr/exo_thigh.STL" /> -->
-    <!-- <xacro:property name="shank_mesh" value="package://yr_lle_sim/urdf/meshes_yr/exo_shank.dae"
-    />
-    <xacro:property name="foot_mesh" value="package://yr_lle_sim/urdf/meshes_yr/exo_foot.dae" /> -->
-    <!-- ======================================================= -->
-    <!-- LINKS                                                   -->
-    <!-- ======================================================= -->
-    <xacro:create_link name="waist_link" m="${waist_m}" l="${waist_l}"
-        w="${waist_w}" h="${waist_h}" mat="${waist_mat}" />
-    <xacro:create_link2 name="l_thigh_link" m="${thigh_m}" l="${thigh_l}" w="${thigh_w}"
-        h="${thigh_h}" o_x="${thigh_w}" o_y="${thigh_w/2}" o_z="${-thigh_l}" o_r="0" o_p="0"
-        o_yaw="${PI}" mat="${thigh_mat}" mesh_filename="${thigh_mesh}" mirror="1" />
-    <xacro:create_link2 name="l_shank_link" m="${shank_m}" l="${shank_l}" w="${shank_w}"
-        h="${shank_h}" o_x="${shank_w}" o_y="${shank_w/2}" o_z="${-shank_l}" o_r="0" o_p="0"
-        o_yaw="${PI}"
-        mat="${shank_mat}" mesh_filename="${shank_mesh}" mirror="1" />
-    <xacro:create_link2 name="l_foot_link" m="${foot_m}" l="${foot_l}" w="${foot_w}"
-        h="${foot_h}" o_x="${-foot_h}" o_y="${foot_w}" o_z="${-foot_l}" o_r="0" o_p="0" o_yaw="0"
-        mat="${foot_mat}"
-        mesh_filename="${foot_mesh}" mirror="-1" />
-    <xacro:create_link2 name="r_thigh_link" m="${thigh_m}" l="${thigh_l}" w="${thigh_w}"
-        h="${thigh_h}" o_x="${-thigh_w}" o_y="${-thigh_w/2}" o_z="${-thigh_l}" o_r="0" o_p="0"
-        o_yaw="0" mat="${thigh_mat}" mesh_filename="${thigh_mesh}" mirror="1" />
-    <xacro:create_link2 name="r_shank_link" m="${shank_m}" l="${shank_l}" w="${shank_w}"
-        h="${shank_h}" o_x="${-shank_w}" o_y="${-shank_w/2}" o_z="${-shank_l}" o_r="0" o_p="0" o_yaw="0"
-        mat="${shank_mat}" mesh_filename="${shank_mesh}" mirror="1" />
-    <xacro:create_link2 name="r_foot_link" m="${foot_m}" l="${foot_l}" w="${foot_w}"
-        h="${foot_h}" o_x="${-foot_h}" o_y="${-foot_w}" o_z="${-foot_l}" o_r="0" o_p="0" o_yaw="0"
-        mat="${foot_mat}"
-        mesh_filename="${foot_mesh}" mirror="1" />
-    <!-- ======================================================= -->
-    <!-- JOINTS                                                  -->
-    <!-- ======================================================= -->
-    <xacro:macro name="create_leg" params="side origin_y">
-        <xacro:create_joint name="${side}_hip_joint" parent="waist_link" child="${side}_thigh_link"
-            origin_x="0" origin_y="${origin_y}" origin_z="0" o_roll="0" o_pitch="0" o_yaw="0"
-            axis_x="0" axis_y="1" axis_z="0"
-            lower_limit="-${PI}" upper_limit="${PI}" effort="100000" velocity="100.0" />
-        <xacro:create_joint name="${side}_kne_joint" parent="${side}_thigh_link"
-            child="${side}_shank_link"
-            origin_x="0" origin_y="0" origin_z="${-thigh_l}" o_roll="0" o_pitch="0" o_yaw="0"
-            axis_x="0" axis_y="1" axis_z="0"
-            lower_limit="-${PI}" upper_limit="${PI}" effort="100000" velocity="100.0" />
-        <xacro:create_joint name="${side}_ank_joint" parent="${side}_shank_link"
-            child="${side}_foot_link"
-            origin_x="0" origin_y="0" origin_z="${-shank_l}" o_roll="0" o_pitch="${-PI/2}" o_yaw="0"
-            axis_x="0" axis_y="1" axis_z="0"
-            lower_limit="-1.75" upper_limit="1.75" effort="1000" velocity="10.0" />
-    </xacro:macro>
-    <xacro:create_leg side="l" origin_y="${waist_w / 2}" />
-    <xacro:create_leg side="r" origin_y="${-waist_w / 2}" />
-    <!-- ======================================================= -->
-    <!-- GAZEBO                                                  -->
-    <!-- ======================================================= -->
-    <gazebo>
-        <plugin name="gazebo_ros2_control" filename="libgazebo_ros2_control.so">
-            <parameters>$(find yr_lle_sim)/config/control.yaml</parameters>
-        </plugin>
-    </gazebo>
-    <ros2_control name="MyRobotHardware" type="system">
-        <hardware>
-            <plugin>gazebo_ros2_control/GazeboSystem</plugin>
-        </hardware>
-        <joint name="l_hip_joint">
-            <commandInterface>effort</commandInterface>
-            <stateInterface>position</stateInterface>
-            <stateInterface>velocity</stateInterface>
-            <stateInterface>effort</stateInterface>
-        </joint>
-        <joint name="l_kne_joint">
-            <commandInterface>effort</commandInterface>
-            <stateInterface>position</stateInterface>
-            <stateInterface>velocity</stateInterface>
-            <stateInterface>effort</stateInterface>
-        </joint>
-    </ros2_control>
-    <xacro:define_gazebo_material link_name="l_thigh_link" r="0.7" g="0.7" b="0.7" a="1" />
-    <xacro:define_gazebo_material link_name="r_thigh_link" r="0.7" g="0.7" b="0.7" a="1" />
-    <xacro:define_gazebo_material link_name="l_shank_link" r="0.8" g="0.8" b="0.8" a="1" />
-    <xacro:define_gazebo_material link_name="r_shank_link" r="0.8" g="0.8" b="0.8" a="1" />
-    <xacro:define_gazebo_material link_name="l_foot_link" r="0.7" g="0.7" b="0.7" a="1" />
-    <xacro:define_gazebo_material link_name="r_foot_link" r="0.7" g="0.7" b="0.7" a="1" />
-    <xacro:define_gazebo_material link_name="stand_base" r="0.4" g="0.4" b="0.4" a="0.5" />
-    <xacro:define_gazebo_material link_name="support_pole" r="0.4" g="0.4" b="0.4" a="0.5" />
-    <xacro:define_gazebo_material link_name="waist_link" r="0.4" g="0.4" b="0.4" a="0.5" />
-    <xacro:macro name="create_leg_transmissions" params="side">
-        <xacro:create_transmission joint_name="${side}_hip_joint" />
-        <xacro:create_transmission joint_name="${side}_kne_joint" />
-        <!-- <xacro:create_transmission joint_name="${side}_ank_joint" /> -->
-    </xacro:macro>
-    <!-- <xacro:create_leg_transmissions side="l" />
-    <xacro:create_leg_transmissions side="r" /> -->
-    <link name="stand_base">
-        <visual>
-            <geometry>
-                <box size="${stand_base_width} ${stand_base_depth} ${stand_base_height}" />
-            </geometry>
-            <material name="black" />
-        </visual>
-        <collision>
-            <geometry>
-                <box size="${stand_base_width} ${stand_base_depth} ${stand_base_height}" />
-            </geometry>
-        </collision>
-        <inertial>
-            <mass value="10.0" /> <!-- Heavier mass to ensure stability -->
-            <inertia ixx="1" iyy="1" izz="1" ixy="0" ixz="0" iyz="0" />
-        </inertial>
-    </link>
-    <!-- Pole Link (Supporting Pole) -->
-    <link name="support_pole">
-        <visual>
-            <geometry>
-                <cylinder length="${pole_height}" radius="${pole_radius}" /> <!-- Variable height for
-                the pole -->
-            </geometry>
-            <material name="silver" />
-        </visual>
-        <collision>
-            <geometry>
-                <cylinder length="${pole_height}" radius="${pole_radius}" />
-            </geometry>
-        </collision>
-        <inertial>
-            <mass value="1.0" />
-            <inertia ixx="0.1" iyy="0.1" izz="0.1" ixy="0" ixz="0" iyz="0" />
-        </inertial>
-    </link>
-    <!-- Joint connecting the stand base to the supporting pole -->
-    <joint name="base_to_pole" type="fixed">
-        <parent link="stand_base" />
-        <child link="support_pole" />
-        <origin xyz="0 0 ${pole_height / 2}" />
-    </joint>
-    <!-- Joint connecting the supporting pole to the waist -->
-    <joint name="pole_to_waist" type="fixed">
-        <parent link="support_pole" />
-        <child link="waist_link" />
-        <origin xyz="0 0 ${pole_height / 2 }" />
-    </joint>
-    <!-- Use the macro to add IMU sensors to specific links -->
-    <xacro:add_imu_sensor link_name="l_thigh_link" />
-    <xacro:add_imu_sensor link_name="r_thigh_link" />
-    <xacro:add_imu_sensor link_name="l_shank_link" />
-    <xacro:add_imu_sensor link_name="r_shank_link" />
-    <xacro:add_imu_sensor link_name="l_foot_link" />
-    <xacro:add_imu_sensor link_name="r_foot_link" />
+  <xacro:include filename="properties.xacro" />
+  <xacro:include filename="macros.xacro" />
+  <xacro:include filename="human_dummy.xacro" />
+  <link name="world"/>
+  <joint name="pole_to_waist" type="fixed">
+    <parent link="world" />
+    <child link="waist_link" />
+    <origin xyz="0 0 0  " />
+  </joint>
+  <xacro:create_link2 name="waist_link" m="${waist_m}" l="${waist_l}" w="${waist_w/2}"
+    h="${waist_h}" o_x="0" o_y="${waist_mesh_w/2 -0.015}" o_z="${-waist_h_offset}" o_r="0"
+    o_p="${-PI}"
+    o_yaw="${-PI}" mat="${waist_mat}" mesh_filename="${waist_mesh}" mirror="1" />
+  <xacro:create_link2 name="l_pel_link" m="${pel_m}" l="${pel_l}" w="${pel_w}"
+    h="${pel_h}" o_x="${pel_x_offset}" o_y="${pel_y_offset}"
+    o_z="${-pel_h_offset}" o_r="0" o_p="0"
+    o_yaw="0" mat="${pel_mat}" mesh_filename="${pel_mesh}" mirror="1" />
+  <xacro:create_link2 name="l_thigh_link" m="${thigh_m}" l="${thigh_l}" w="${thigh_w}"
+    h="${thigh_h}" o_x="${thigh_w}" o_y="${thigh_w/2}" o_z="${-thigh_l}" o_r="0" o_p="0"
+    o_yaw="${PI}" mat="${thigh_mat}" mesh_filename="${thigh_mesh}" mirror="1" />
+  <xacro:create_link2 name="l_shank_link" m="${shank_m}" l="${shank_l}" w="${shank_w}"
+    h="${shank_h}" o_x="${shank_w}" o_y="${shank_w/2}" o_z="${-shank_l}" o_r="0" o_p="0"
+    o_yaw="${PI}"
+    mat="${shank_mat}" mesh_filename="${shank_mesh}" mirror="1" />
+  <xacro:create_link2 name="l_foot_link" m="${foot_m}" l="${foot_h}" w="${foot_w}"
+    h="${foot_h}" o_x="${-foot_h}" o_y="${foot_w}" o_z="${-foot_l}" o_r="0" o_p="0" o_yaw="0"
+    mat="${foot_mat}"
+    mesh_filename="${foot_mesh}" mirror="-1" />
+  <xacro:create_link2 name="r_pel_link" m="${pel_m}" l="${pel_l}" w="${pel_w}"
+    h="${pel_h}" o_x="${pel_x_offset}" o_y="${pel_y_offset}"
+    o_z="${-pel_h_offset}" o_r="0" o_p="0"
+    o_yaw="0" mat="${pel_mat}" mesh_filename="${pel_mesh}" mirror="1" />
+  <xacro:create_link2 name="r_thigh_link" m="${thigh_m}" l="${thigh_l}" w="${thigh_w}"
+    h="${thigh_h}" o_x="${-thigh_w}" o_y="${-thigh_w/2}" o_z="${-thigh_l}" o_r="0" o_p="0"
+    o_yaw="0" mat="${thigh_mat}" mesh_filename="${thigh_mesh}" mirror="1" />
+  <xacro:create_link2 name="r_shank_link" m="${shank_m}" l="${shank_l}" w="${shank_w}"
+    h="${shank_h}" o_x="${-shank_w}" o_y="${-shank_w/2}" o_z="${-shank_l}" o_r="0" o_p="0" o_yaw="0"
+    mat="${shank_mat}" mesh_filename="${shank_mesh}" mirror="1" />
+  <xacro:create_link2 name="r_foot_link" m="${foot_m}" l="${foot_l}" w="${foot_w}"
+    h="${foot_h}" o_x="${-foot_h}" o_y="${-foot_w}" o_z="${-foot_l}" o_r="0" o_p="0" o_yaw="0"
+    mat="${foot_mat}"
+    mesh_filename="${foot_mesh}" mirror="1" />
+  <!-- ======================================================= -->
+  <!-- JOINTS                                                  -->
+  <!-- ======================================================= -->
+  <xacro:macro name="create_leg" params="side origin_y o_roll hip_y_offset">
+    <xacro:create_joint2 name="yr_${side}_pel_joint" parent="waist_link"
+      child="${side}_pel_link" origin_x="0" origin_y="${origin_y}"
+      origin_z="0" o_roll="0"
+      o_pitch="0" o_yaw="${-PI}"
+      axis_x="1" axis_y="0" axis_z="0"
+      lower_limit="-3.14" upper_limit="3.14" effort="1000" velocity="10.0" />
+    <xacro:create_joint2 name="yr_${side}_hip_joint" parent="${side}_pel_link"
+      child="${side}_thigh_link"
+      origin_x="${-pel_l}" origin_y="${hip_y_offset}" origin_z="${-pel_h}" o_roll="${o_roll}"
+      o_pitch="0" o_yaw="${-PI}"
+      axis_x="0" axis_y="1" axis_z="0"
+      lower_limit="-${PI}" upper_limit="${PI}" effort="100000" velocity="100.0" />
+    <xacro:create_joint2 name="yr_${side}_kne_joint" parent="${side}_thigh_link"
+      child="${side}_shank_link"
+      origin_x="0" origin_y="0" origin_z="${-thigh_l}" o_roll="0" o_pitch="0" o_yaw="0"
+      axis_x="0" axis_y="1" axis_z="0"
+      lower_limit="-${PI}" upper_limit="${PI}" effort="100000" velocity="100.0" />
+    <xacro:create_joint2 name="yr_${side}_ank_joint" parent="${side}_shank_link"
+      child="${side}_foot_link"
+      origin_x="0" origin_y="0" origin_z="${-shank_l}" o_roll="0" o_pitch="0" o_yaw="0"
+      axis_x="0" axis_y="1" axis_z="0"
+      lower_limit="-1.75" upper_limit="1.75" effort="1000" velocity="10.0" />
+  </xacro:macro>
+  <xacro:create_leg side="l" origin_y="${(abduction_motor_distance) / 2}" o_roll="${-PI/2}"
+    hip_y_offset="${-pel_w/2}" />
+  <xacro:create_leg side="r" origin_y="${-(abduction_motor_distance) / 2}" o_roll="${PI/2}"
+    hip_y_offset="${pel_w/2}" />
+  <link name="human_waist_link">
+    <visual>
+      <origin xyz="0 0 ${-human_waist_h/2}" rpy="0 0 0" />
+      <geometry>
+        <box size="${human_waist_l} ${human_waist_w} ${human_waist_h}" />
+      </geometry>
+      <material name="black" />
+    </visual>
+    <collision>
+      <origin xyz="0 0 ${-human_waist_h/2}" rpy="0 0 0" />
+      <geometry>
+        <box size="${human_waist_l} ${human_waist_w} ${human_waist_h}" />
+      </geometry>
+    </collision>
+    <inertial>
+      <origin xyz="0 0 ${-human_waist_h/2}" rpy="0 0 0" />
+      <mass value="${human_waist_weight}" />
+      <inertia
+        ixx="${human_waist_weight / 12.0 * (human_waist_w**2 + human_waist_h**2)}"
+        iyy="${human_waist_weight / 12.0 * (human_waist_l**2 + human_waist_h**2)}"
+        izz="${human_waist_weight / 12.0 * (human_waist_l**2 + human_waist_w**2)}"
+        ixy="0"
+        ixz="0"
+        iyz="0" />
+    </inertial>
+  </link>
+  <joint name="human_waist_link_joint" type="fixed">
+    <parent link="waist_link" />
+    <child link="human_waist_link" />
+    <origin xyz="${human_waist_l/2} 0 ${human_waist_h}" rpy="0 0 0" />
+  </joint>
+  <xacro:create_human_leg side="l" />
+  <xacro:create_human_leg side="r" />
+  <ros2_control name="GazeboSystem" type="system">
+    <hardware>
+      <plugin>gazebo_ros2_control/GazeboSystem</plugin>
+    </hardware>
+    <joint name="human_l_thigh_abduction_joint">
+      <command_interface name="effort">
+        <param name="min">-1000</param>
+        <param name="max">1000</param>
+      </command_interface>
+      <state_interface name="position" />
+      <state_interface name="velocity" />
+      <state_interface name="effort" />
+    </joint>
+    <joint name="human_l_thigh_flexion_joint">
+      <command_interface name="effort">
+        <param name="min">-1000</param>
+        <param name="max">1000</param>
+      </command_interface>
+      <state_interface name="position" />
+      <state_interface name="velocity" />
+      <state_interface name="effort" />
+    </joint>
+    <joint name="human_l_thigh_rotation_joint">
+      <command_interface name="effort">
+        <param name="min">-1000</param>
+        <param name="max">1000</param>
+      </command_interface>
+      <state_interface name="position" />
+      <state_interface name="velocity" />
+      <state_interface name="effort" />
+    </joint>
+    <joint name="human_l_kne_joint">
+      <command_interface name="effort">
+        <param name="min">-1000</param>
+        <param name="max">1000</param>
+      </command_interface>
+      <state_interface name="position" />
+      <state_interface name="velocity" />
+      <state_interface name="effort" />
+    </joint>
+    <joint name="human_l_ank_joint">
+      <command_interface name="effort">
+        <param name="min">-1000</param>
+        <param name="max">1000</param>
+      </command_interface>
+      <state_interface name="position" />
+      <state_interface name="velocity" />
+      <state_interface name="effort" />
+    </joint>
+    <joint name="human_r_thigh_abduction_joint">
+      <command_interface name="effort">
+        <param name="min">-1000</param>
+        <param name="max">1000</param>
+      </command_interface>
+      <state_interface name="position" />
+      <state_interface name="velocity" />
+      <state_interface name="effort" />
+    </joint>
+    <joint name="human_r_thigh_flexion_joint">
+      <command_interface name="effort">
+        <param name="min">-1000</param>
+        <param name="max">1000</param>
+      </command_interface>
+      <state_interface name="position" />
+      <state_interface name="velocity" />
+      <state_interface name="effort" />
+    </joint>
+    <joint name="human_r_thigh_rotation_joint">
+      <command_interface name="effort">
+        <param name="min">-1000</param>
+        <param name="max">1000</param>
+      </command_interface>
+      <state_interface name="position" />
+      <state_interface name="velocity" />
+      <state_interface name="effort" />
+    </joint>
+    <joint name="human_r_kne_joint">
+      <command_interface name="effort">
+        <param name="min">-1000</param>
+        <param name="max">1000</param>
+      </command_interface>
+      <state_interface name="position" />
+      <state_interface name="velocity" />
+      <state_interface name="effort" />
+    </joint>
+    <joint name="human_r_ank_joint">
+      <command_interface name="effort">
+        <param name="min">-1000</param>
+        <param name="max">1000</param>
+      </command_interface>
+      <state_interface name="position" />
+      <state_interface name="velocity" />
+      <state_interface name="effort" />
+    </joint>
+<!--  -->
+    <!-- Yr Bot Joint Control -->
+<!--  -->
+    <joint name="yr_l_pel_joint">
+      <command_interface name="effort">
+        <param name="min">-1000</param>
+        <param name="max">1000</param>
+      </command_interface>
+      <state_interface name="position" />
+      <state_interface name="velocity" />
+      <state_interface name="effort" />
+    </joint>
+    <joint name="yr_l_hip_joint">
+      <command_interface name="effort">
+        <param name="min">-1000</param>
+        <param name="max">1000</param>
+      </command_interface>
+      <state_interface name="position" />
+      <state_interface name="velocity" />
+      <state_interface name="effort" />
+    </joint>
+    <joint name="yr_l_kne_joint">
+      <command_interface name="effort">
+        <param name="min">-1000</param>
+        <param name="max">1000</param>
+      </command_interface>
+      <state_interface name="position" />
+      <state_interface name="velocity" />
+      <state_interface name="effort" />
+    </joint>
+    <joint name="yr_l_ank_joint">
+      <command_interface name="effort">
+        <param name="min">-1000</param>
+        <param name="max">1000</param>
+      </command_interface>
+      <state_interface name="position" />
+      <state_interface name="velocity" />
+      <state_interface name="effort" />
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
File: src/yr_lle_sim/urdf/properties.xacro (robot description, xacro)
@@ -12,17 +12,19 @@
         <color rgba="0.8 0.8 1 ${alpha}" />
     </material>
+    <xacro:property name="abduction_motor_distance" value="0.35" />
     <xacro:property name="waist_m" value="2.0" />
     <xacro:property name="waist_l" value="0.05" />
     <xacro:property name="waist_h" value="0.05" />
     <xacro:property name="waist_mat" value="silver" />
-    <xacro:property name="waist_mesh_w" value="0.42" />
+    <xacro:property name="waist_mesh_w" value="0.45" />
     <xacro:property name="waist_w" value="${waist_mesh_w}" />
     <xacro:property name="waist_h_offset" value="0.062" />
+    <xacro:property name="pel_joints_dist" value="0.4" />
     <xacro:property name="waist_mesh"
         value="file://$(find yr_lle_sim)/urdf/meshes_yr/waist_center.STL" />
     <xacro:property name="pel_m" value="1.0" />
-    <xacro:property name="pel_l" value="0.0" />
-    <xacro:property name="pel_w" value="0.0" />
-    <xacro:property name="pel_h" value="0.0" />
+    <xacro:property name="pel_l" value="0.1" />
+    <xacro:property name="pel_w" value="0.05" />
+    <xacro:property name="pel_h" value="0.1" />
     <xacro:property name="pel_mat" value="silver" />
     <xacro:property name="pel_x_offset" value="-0.09" />
@@ -30,5 +32,5 @@
     <xacro:property name="pel_h_offset" value="0.088" />
     <xacro:property name="pel_mesh"
-        value="file://$(find yr_lle_sim)/urdf/meshes_yr/orig.waist_corner_bracket.STL" />
+        value="file://$(find yr_lle_sim)/urdf/meshes_yr/waist_corner_bracket.STL" />
     <xacro:property name="thigh_m" value="1.5" />
     <xacro:property name="thigh_l" value="0.468" />
@@ -54,3 +56,14 @@
     <xacro:property name="shank_mesh" value="file://$(find yr_lle_sim)/urdf/meshes_yr/exo_shank.STL" />
     <xacro:property name="foot_mesh" value="file://$(find yr_lle_sim)/urdf/meshes_yr/exo_foot.STL" />
+    <!-- Human Boday Paramters -->
+    <xacro:property name="human_thigh_r" value="0.075" />
+    <xacro:property name="human_shank_r" value="0.056" />
+    <xacro:property name="human_waist_l" value="0.1" />
+    <xacro:property name="human_waist_w" value="0.35" />
+    <xacro:property name="human_waist_h" value="0.4" />
+    <xacro:property name="human_weight" value="70" />
+    <xacro:property name="human_waist_weight" value="${human_weight*0.842}" />
+    <xacro:property name="human_thigh_weight" value="${human_weight*0.1}" />
+    <xacro:property name="human_shank_weight" value="${human_weight*0.05}" />
+    <xacro:property name="human_foot_weight" value="${human_weight*0.015}" />
 </robot>
