Commit message: interface ready

File: src/yr_lle_sim/urdf/macros.xacro (robot description, xacro)
@@ -104,4 +104,51 @@
         </link>
     </xacro:macro>
+    <xacro:macro name="create_link3"
+        params="name m l w h o_x o_y o_z o_r o_p o_yaw mat mesh_filename mirror">
+        <link name="${name}">
+            <collision>
+                <origin xyz="0 0 ${-l/2}" rpy="0 0 0" />
+                <geometry>
+                    <box size="${h} ${w} ${l*0.6}" />
+                </geometry>
+            </collision>
+            <visual>
+                <!-- <xacro:if value="${use_mesh}">
+                    <mesh_filename="" />
+                </xacro:if> -->
+                <!-- <xacro:property name="o_rpy_parts" value="split(o_rpy)" />
+                <xacro:property name="o_yaw" value="${(o_rpy_parts[2])}" /> -->
+                <xacro:if value="${mesh_filename != ''}">
+                    <!-- <origin xyz="0 0 0" rpy="0 0 ${-PI}" /> -->
+                    <!-- <origin xyz="${-h} ${-w/2} ${-l}" rpy="${PI/2} 0 ${PI/2 + float(o_yaw)}" /> -->
+                    <origin xyz="${o_x} ${o_y} ${o_z}" rpy="${PI/2} 0 ${PI/2 + o_yaw}" />
+                </xacro:if>
+                <xacro:unless value="${mesh_filename != ''}">
+                    <origin xyz="0 0 ${-l/2}" rpy="0 0 ${-PI}" />
+                </xacro:unless>
+                <geometry>
+                    <xacro:if value="${mesh_filename != ''}">
+                        <mesh filename="${mesh_filename}"
+                            scale="${mirror*mesh_scale} ${mesh_scale} ${mesh_scale}" />
+                    </xacro:if>
+                    <xacro:unless value="${mesh_filename != ''}">
+                        <box size="${h} ${w} ${l}" />
+                    </xacro:unless>
+                </geometry>
+                <origin xyz="0 0 ${-l/2}" rpy="0 0 0" />
+                <material name="${mat}" />
+            </visual>
+            <inertial>
+                <origin xyz="0 0 ${-l/2}" rpy="0 0 0" />
+                <mass value="${m}" />
+                <inertia
+                    ixx="${m / 12.0 * (w*w + l*l)}"
+                    ixy="0.0" ixz="0.0"
+                    iyy="${m / 12.0 * (h*h + l*l)}"
+                    iyz="0.0"
+                    izz="${m / 12.0 * (h*h + w*w)}" />
+            </inertial>
+        </link>
+    </xacro:macro>
     <!-- ======================================================= -->
     <!-- JOINTS                                                  -->
@@ -149,4 +196,9 @@
     <xacro:macro name="define_gazebo_material" params="link_name r g b a">
         <gazebo reference="${link_name}">
+            <mu1>3</mu1>
+            <mu2>3</mu2>
+            <kp  value="1000000.0"/>
+            <kd  value="1000.0"/>
+            <self_collide>0</self_collide>
             <material>Gazebo/White</material>
             <visual>
@@ -158,4 +210,16 @@
                 </material>
             </visual>
+            <!-- <collision>
+                <surface>
+                    <friction>
+                        <ode>
+                            <mu1>2</mu1>
+                            <mu2>2</mu2>
+                            <kp value="1000000.0" />
+                            <kd value="1000.0" />
+                        </ode>
+                    </friction>
+                </surface>
+            </collision> -->
         </gazebo>
     </xacro:macro>

File: src/yr_lle_sim/urdf/model_gazebo.xacro (robot description, xacro)
@@ -204,76 +204,92 @@
     <!-- Yr Bot Joint Control -->
 <!--  -->
-    <joint name="yr_l_pel_joint">
-      <command_interface name="effort">
-        <param name="min">-1000</param>
-        <param name="max">1000</param>
-      </command_interface>
-      <state_interface name="position" />
-      <state_interface name="velocity" />
-      <state_interface name="effort" />
-    </joint>
-    <joint name="yr_l_hip_joint">
-      <command_interface name="effort">
-        <param name="min">-1000</param>
-        <param name="max">1000</param>
-      </command_interface>
-      <state_interface name="position" />
-      <state_interface name="velocity" />
-      <state_interface name="effort" />
-    </joint>
-    <joint name="yr_l_kne_joint">
-      <command_interface name="effort">
-        <param name="min">-1000</param>
-        <param name="max">1000</param>
-      </command_interface>
-      <state_interface name="position" />
-      <state_interface name="velocity" />
-      <state_interface name="effort" />
-    </joint>
-    <joint name="yr_l_ank_joint">
-      <command_interface name="effort">
-        <param name="min">-1000</param>
-        <param name="max">1000</param>
-      </command_interface>
-      <state_interface name="position" />
-      <state_interface name="velocity" />
-      <state_interface name="effort" />
-    </joint>
-    <joint name="yr_r_pel_joint">
-      <command_interface name="effort">
-        <param name="min">-1000</param>
-        <param name="max">1000</param>
-      </command_interface>
-      <state_interface name="position" />
-      <state_interface name="velocity" />
-      <state_interface name="effort" />
-    </joint>
-    <joint name="yr_r_hip_joint">
-      <command_interface name="effort">
-        <param name="min">-1000</param>
-        <param name="max">1000</param>
-      </command_interface>
-      <state_interface name="position" />
-      <state_interface name="velocity" />
-      <state_interface name="effort" />
-    </joint>
-    <joint name="yr_r_kne_joint">
-      <command_interface name="effort">
-        <param name="min">-1000</param>
-        <param name="max">1000</param>
-      </command_interface>
-      <state_interface name="position" />
-      <state_interface name="velocity" />
-      <state_interface name="effort" />
-    </joint>
-    <joint name="yr_r_ank_joint">
-      <command_interface name="effort">
-        <param name="min">-1000</param>
-        <param name="max">1000</param>
-      </command_interface>
-      <state_interface name="position" />
-      <state_interface name="velocity" />
-      <state_interface name="effort" />
-    </joint>
+<joint name="yr_l_pel_joint">
+  <command_interface name="position">
+    <param name="min">-3.14</param>
+    <param name="max">3.14</param>
+  </command_interface>
+  <state_interface name="position">
+    <param name="initial_value">1.0</param>
+  </state_interface>
+  <state_interface name="velocity" />
+  <state_interface name="effort" />
+</joint>
+<joint name="yr_l_hip_joint">
+  <command_interface name="position">
+    <param name="min">-3.14</param>
+    <param name="max">3.14</param>
+  </command_interface>
+  <state_interface name="position">
+    <param name="initial_value">1.0</param>
+  </state_interface>
+  <state_interface name="velocity" />
+  <state_interface name="effort" />
+</joint>
+<joint name="yr_l_kne_joint">
+  <command_interface name="position">
+    <param name="min">-3.14</param>
+    <param name="max">3.14</param>
+  </command_interface>
+  <state_interface name="position">
+    <param name="initial_value">1.0</param>
+  </state_interface>
+  <state_interface name="velocity" />
+  <state_interface name="effort" />
+</joint>
+<joint name="yr_l_ank_joint">
+  <command_interface name="position">
+    <param name="min">-3.14</param>
+    <param name="max">3.14</param>
+  </command_interface>
+  <state_interface name="position">
+    <param name="initial_value">1.0</param>
+  </state_interface>
+  <state_interface name="velocity" />
+  <state_interface name="effort" />
+</joint>
+<joint name="yr_r_pel_joint">
+  <command_interface name="position">
+    <param name="min">-3.14</param>
+    <param name="max">3.14</param>
+  </command_interface>
+  <state_interface name="position">
+    <param name="initial_value">1.0</param>
+  </state_interface>
+  <state_interface name="velocity" />
+  <state_interface name="effort" />
+</joint>
+<joint name="yr_r_hip_joint">
+  <command_interface name="position">
+    <param name="min">-3.14</param>
+    <param name="max">3.14</param>
+  </command_interface>
+  <state_interface name="position">
+    <param name="initial_value">1.0</param>
+  </state_interface>
+  <state_interface name="velocity" />
+  <state_interface name="effort" />
+</joint>
+<joint name="yr_r_kne_joint">
+  <command_interface name="position">
+    <param name="min">-3.14</param>
+    <param name="max">3.14</param>
+  </command_interface>
+  <state_interface name="position">
+    <param name="initial_value">1.0</param>
+  </state_interface>
+  <state_interface name="velocity" />
+  <state_interface name="effort" />
+</joint>
+<joint name="yr_r_ank_joint">
+  <command_interface name="position">
+    <param name="min">-3.14</param>
+    <param name="max">3.14</param>
+  </command_interface>
+  <state_interface name="position">
+    <param name="initial_value">1.0</param>
+  </state_interface>
+  <state_interface name="velocity" />
+  <state_interface name="effort" />
+</joint>
   </ros2_control>
   <gazebo>

File: src/yr_lle_sim/urdf/properties.xacro (robot description, xacro)
@@ -46,5 +46,5 @@
     <xacro:property name="foot_l" value="0.15" />
     <xacro:property name="foot_w" value="0.08" />
-    <xacro:property name="foot_h" value="0.10" />
+    <xacro:property name="foot_h" value="0.1" />
     <xacro:property name="foot_mat" value="silver" />
     <xacro:property name="stand_base_width" value="0.5" />
@@ -59,11 +59,19 @@
     <xacro:property name="human_thigh_r" value="0.075" />
     <xacro:property name="human_shank_r" value="0.056" />
-    <xacro:property name="human_waist_l" value="0.1" />
+    <xacro:property name="human_waist_l" value="0.25" />
     <xacro:property name="human_waist_w" value="0.35" />
     <xacro:property name="human_waist_h" value="0.4" />
-    <xacro:property name="human_weight" value="70" />
+    <xacro:property name="human_weight" value="75" />
     <xacro:property name="human_waist_weight" value="${human_weight*0.842}" />
     <xacro:property name="human_thigh_weight" value="${human_weight*0.1}" />
     <xacro:property name="human_shank_weight" value="${human_weight*0.05}" />
     <xacro:property name="human_foot_weight" value="${human_weight*0.015}" />
+    <xacro:property name="yr_l_pel_joint_val" value="${-PI/2}" />
+    <xacro:property name="yr_l_hip_joint_val" value="${-PI/4}" />
+    <xacro:property name="yr_l_kne_joint_val" value="${PI/2}" />
+    <xacro:property name="yr_l_ank_joint_val" value="${-PI/4}" />
+    <xacro:property name="yr_r_pel_joint_val" value="${PI/2}" />
+    <xacro:property name="yr_r_hip_joint_val" value="${-PI/4}" />
+    <xacro:property name="yr_r_kne_joint_val" value="${PI/2}" />
+    <xacro:property name="yr_r_ank_joint_val" value="${-PI/4}" />
 </robot>
